File: Kicad_design/close_door.kicad_pcb (KiCad board)
At the start: 2 copper layers, 94 x 43.2 mm, 56 parts, among them Q1 AO3400A, SW1 my_SW_Reed_SPDT, U1 SN74LVC2G02DCTR, U2 LTC6993IS6-3, U3 LTC6993IS6-3, U5 SMTU2450N-LF, U6 TLC556CDR

Commit message: V1.7
Parts:
- C14, C16: footprint PCM_JLCPCB:C_0603 -> Capacitor_SMD:C_0603_1608Metric
- Q1: footprint PCM_JLCPCB:Q_SOT-23 -> Package_TO_SOT_SMD:SOT-23
- R2, R9: footprint PCM_JLCPCB:R_0805 -> Resistor_SMD:R_0805_2012Metric
- U5: footprint Battery:BatteryHolder_Renata_SMTU2032-LF_1x2032 -> Nadavs_Library:SMTU2450N1LF
- moved H4 48.3 mm to (97.8, 135.9)
- moved H2 48.3 mm to (97.8, 102.9)
- moved FID1 34.1 mm to (123.2, 102.9)
- moved LS1 32.0 mm to (111.8, 111.8)
- moved C10 27.1 mm to (115.6, 102.9), turned to 0 degrees
- moved R2 25.6 mm to (116.8, 120.7), turned to 0 degrees
- moved U5 24.5 mm to (139.7, 118.1), turned to -90 degrees
- moved Q1 21.2 mm to (121.9, 115.9)
- moved R9 15.2 mm to (121.9, 108.0)
- moved D2 14.8 mm to (123.2, 133.3), turned to 0 degrees
- moved TP7 13.3 mm to (113.0, 120.7)
- moved C16 13.1 mm to (121.9, 136.7)
- moved C14 11.9 mm to (124.5, 136.7)
- moved C9 10.6 mm to (108.0, 121.9), turned to 180 degrees
- moved C8 10.5 mm to (116.8, 134.6)
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Routing:
- net VCC: track 239.4 -> 204.6 mm
- net beeps: track 33.1 -> 16.3 mm, vias 0 -> 2
- net Net-(C7-Pad1): track 19.6 -> 10.3 mm, vias 2 -> 0
- net GND: track 41.0 -> 35.0 mm, vias 31 -> 38
- net Net-(U6B-TR): track 29.9 -> 24.8 mm, vias 1 -> 0
- net Net-(Q1-D): track 21.9 -> 17.3 mm
- net Net-(U2-OUT): track 16.8 -> 12.4 mm
- net beep_length: track 37.7 -> 34.7 mm
- net Net-(U3-OUT): track 26.0 -> 24.3 mm
- net Net-(U6A-TR): track 19.4 -> 21.0 mm
- net Net-(Q1-G): track 4.50 -> 5.79 mm
- net Net-(U6B-CV): track 8.04 -> 7.37 mm
Other:
- board size 94 x 43.2 mm -> 97.8 x 43.2 mm
- board text added: "close the door! V1.7"
- board text removed: "close the door! V1.6"
