File: Kicad_design/close_door.kicad_sch (KiCad schematic)
At the start: 56 parts, among them Q1 AO3400A, SW1 my_SW_Reed_SPDT, U1 SN74LVC2G02DCTR, U2 LTC6993IS6-3, U3 LTC6993IS6-3, U5 SMTU2450N-LF, U6 TLC556CDR

Commit message: V1.7
Parts:
- C14, C16: footprint PCM_JLCPCB:C_0603 -> Capacitor_SMD:C_0603_1608Metric
- Q1: footprint PCM_JLCPCB:Q_SOT-23 -> Package_TO_SOT_SMD:SOT-23
- R2, R9: footprint PCM_JLCPCB:R_0805 -> Resistor_SMD:R_0805_2012Metric
- U5: footprint Battery:BatteryHolder_Renata_SMTU2032-LF_1x2032 -> Nadavs_Library:SMTU2450N1LF
Changed lines of the file:
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@@
 			)
 		)
-		(property "Footprint" "PCM_JLCPCB:R_0805"
+		(property "Footprint" "Resistor_SMD:R_0805_2012Metric"
 			(at 241.3 151.638 90)
 			(effects
@@
 			)
 		)
-		(property "Footprint" "PCM_JLCPCB:Q_SOT-23"
+		(property "Footprint" "Package_TO_SOT_SMD:SOT-23"
 			(at 252.222 149.86 90)
 			(effects
@@
 			)
 		)
-		(property "Footprint" "PCM_JLCPCB:C_0603"
+		(property "Footprint" "Capacitor_SMD:C_0603_1608Metric"
 			(at 197.612 153.67 90)
 			(effects
@@
 			)
 		)
-		(property "Footprint" "PCM_JLCPCB:C_0603"
+		(property "Footprint" "Capacitor_SMD:C_0603_1608Metric"
 			(at 206.502 153.67 90)
 			(effects
@@
 			)
 		)
-		(property "Footprint" "PCM_JLCPCB:R_0805"
+		(property "Footprint" "Resistor_SMD:R_0805_2012Metric"
 			(at 247.142 130.81 90)
 			(effects
@@
 			)
 		)
-		(property "Footprint" "Battery:BatteryHolder_Renata_SMTU2032-LF_1x2032"
+		(property "Footprint" "Nadavs_Library:SMTU2450N1LF"
 			(at 100.33 134.29 0)
 			(effects
